Commit message: use base and roof instead of left and right

File: pmb3_description/urdf/base/base_pmb3_calib.urdf.xacro (robot description, xacro)
@@ -5,9 +5,9 @@
 -->
 <robot xmlns:xacro="http://ros.org/wiki/xacro">
-  <xacro:property name="left_rgbd_z" value="0.164028397812952"/>
-  <xacro:property name="left_rgbd_R" value="180.0"/>
-  <xacro:property name="left_rgbd_P" value="0.0"/>
-  <xacro:property name="right_rgbd_z" value="0.147644299790751"/>
-  <xacro:property name="right_rgbd_R" value="21.612"/>
-  <xacro:property name="right_rgbd_P" value="29.904"/>
+  <xacro:property name="base_rgbd_z" value="0.147644299790751"/>
+  <xacro:property name="base_rgbd_R" value="21.612"/>
+  <xacro:property name="base_rgbd_P" value="29.904"/>
+  <xacro:property name="roof_rgbd_z" value="0.164028397812952"/>
+  <xacro:property name="roof_rgbd_R" value="180.0"/>
+  <xacro:property name="roof_rgbd_P" value="0.0"/>
 </robot>

File: pmb3_description/urdf/base/base_sensors.urdf.xacro (robot description, xacro)
@@ -10,10 +10,6 @@
   <xacro:include filename="$(find pmb3_description)/urdf/base/base.urdf.xacro"/>
   <xacro:include filename="$(find pmb3_description)/urdf/sensors/sick_nanoscan3_laser.urdf.xacro"/>
-  <xacro:include filename="$(find pmb2_description)/urdf/sensors/hokuyo_urg_04lx_ug01_laser.urdf.xacro"/>
-  <xacro:include filename="$(find pmb2_description)/urdf/sensors/sick_tim551_laser.urdf.xacro"/>
-  <xacro:include filename="$(find pmb2_description)/urdf/sensors/sick_tim561_laser.urdf.xacro"/>
   <xacro:include filename="$(find pmb2_description)/urdf/sensors/sick_tim571_laser.urdf.xacro"/>
   <xacro:include filename="$(find realsense2_description)/urdf/_d435.urdf.xacro" />
-  <xacro:include filename="$(find stockbot_description)/urdf/sensors/structure_sensor.urdf.xacro"/>
   <xacro:include filename="$(find pmb3_description)/urdf/deg_to_rad.xacro"/>
   <!-- Laser characteristics -->
@@ -25,34 +21,13 @@
   <xacro:property name="calibration_path" value="$(optenv pmb3_description_calibration_path ${default_calibration_path})"/>
   <xacro:include filename="${calibration_path}/urdf/base/base_pmb3_calib.urdf.xacro"/>
-  <xacro:property name="left_rgbd_x" value="0.249110911156978"/>
-  <xacro:property name="left_rgbd_y" value="0.117678395770306"/>
-  <xacro:property name="left_rgbd_Y" value="-10.0"/>
-  <xacro:property name="right_rgbd_x" value="0.260434779504343"/>
-  <xacro:property name="right_rgbd_y" value="-0.112224592786096"/>
-  <xacro:property name="right_rgbd_Y" value="3.738"/>
+  <xacro:property name="base_rgbd_x" value="0.260434779504343"/>
+  <xacro:property name="base_rgbd_y" value="-0.112224592786096"/>
+  <xacro:property name="base_rgbd_Y" value="3.738"/>
+  <xacro:property name="roof_rgbd_x" value="0.249110911156978"/>
+  <xacro:property name="roof_rgbd_y" value="0.117678395770306"/>
+  <xacro:property name="roof_rgbd_Y" value="-10.0"/>
   <!-- Laser model can be: false, hokuyo, sick-551, sick-561, sick-571, sick-nanoscan-3 -->
   <!-- Camera model can be: false, realsense-d435, structure -->
   <xacro:macro name="base_sensors" params=" name laser_model:=sick-nanoscan-3 camera_model:=realsense-d435">
-    <xacro:if value="${laser_model == 'hokuyo'}">
-      <!-- Laser -->
-      <!-- Theoretic FOV = 220 -->
-      <xacro:hokuyo_urg_04lx_ug01_laser name="${name}_laser" parent="${name}" ros_topic="scan_raw" update_rate="10" min_angle="${-110 * deg_to_rad}" max_angle="${110 * deg_to_rad}" >
-        <origin xyz="${base_laser_x} ${base_laser_y} ${base_laser_z}" rpy="0 0 0" />
-      </xacro:hokuyo_urg_04lx_ug01_laser>
-    </xacro:if>
-    <xacro:if value="${laser_model == 'sick-551'}">
-      <!-- Laser -->
-      <!-- Theoretic FOV = 220 -->
-      <xacro:sick_tim551_laser name="${name}_laser" parent="${name}" ros_topic="scan_raw" update_rate="10" min_angle="${-110 * deg_to_rad}" max_angle="${110 * deg_to_rad}" >
-        <origin xyz="${base_laser_x} ${base_laser_y} ${base_laser_z}" rpy="0 0 0" />
-      </xacro:sick_tim551_laser>
-    </xacro:if>
-    <xacro:if value="${laser_model == 'sick-561'}">
-      <!-- Laser -->
-      <!-- Theoretic FOV = 220 -->
-      <xacro:sick_tim561_laser name="${name}_laser" parent="${name}" ros_topic="scan_raw" update_rate="10" min_angle="${-110 * deg_to_rad}" max_angle="${110 * deg_to_rad}" >
-        <origin xyz="${base_laser_x} ${base_laser_y} ${base_laser_z}" rpy="0 0 0" />
-      </xacro:sick_tim561_laser>
-    </xacro:if>
     <xacro:if value="${laser_model == 'sick-571'}">
       <!-- Laser -->
@@ -65,24 +40,16 @@
       <!-- Laser -->
       <!-- Theoretic FOV = 275 (using 240) -->
-      <xacro:sick_tim571_laser name="${name}_laser" parent="${name}" ros_topic="scan_raw" update_rate="15" min_angle="${-120 * deg_to_rad}" max_angle="${120 * deg_to_rad}" >
+      <xacro:sick_nanoscan3_laser name="${name}_laser" parent="${name}" ros_topic="scan_raw" update_rate="15" min_angle="${-120 * deg_to_rad}" max_angle="${120 * deg_to_rad}" >
         <origin xyz="${base_laser_x} ${base_laser_y} ${base_laser_z}" rpy="0 0 0" />
-      </xacro:sick_tim571_laser>
+      </xacro:sick_nanoscan3_laser>
     </xacro:if>
     <!-- RGBD camera -->
     <xacro:if value="${camera_model == 'realsense-d435'}">
-      <xacro:sensor_d435 name="left_rgbd_camera" parent="${name}_link" topics_ns="left_rgbd_camera">
-        <origin xyz="${left_rgbd_x} ${left_rgbd_y} ${left_rgbd_z}" rpy="${left_rgbd_R * deg_to_rad} ${left_rgbd_P * deg_to_rad} ${left_rgbd_Y * deg_to_rad}"/>
+      <xacro:sensor_d435 name="roof_rgbd_camera" parent="${name}_link" topics_ns="roof_rgbd_camera">
+        <origin xyz="${roof_rgbd_x} ${roof_rgbd_y} ${roof_rgbd_z}" rpy="${roof_rgbd_R * deg_to_rad} ${roof_rgbd_P * deg_to_rad} ${roof_rgbd_Y * deg_to_rad}"/>
       </xacro:sensor_d435>
-      <xacro:sensor_d435 name="right_rgbd_camera" parent="${name}_link" topics_ns="right_rgbd_camera">
-        <origin xyz="${right_rgbd_x} ${right_rgbd_y} ${right_rgbd_z}" rpy="${right_rgbd_R * deg_to_rad} ${right_rgbd_P * deg_to_rad} ${right_rgbd_Y * deg_to_rad}"/>
+      <xacro:sensor_d435 name="base_rgbd_camera" parent="${name}_link" topics_ns="base_rgbd_camera">
+        <origin xyz="${base_rgbd_x} ${base_rgbd_y} ${base_rgbd_z}" rpy="${base_rgbd_R * deg_to_rad} ${base_rgbd_P * deg_to_rad} ${base_rgbd_Y * deg_to_rad}"/>
       </xacro:sensor_d435>
-    </xacro:if>
-    <xacro:if value="${camera_model == 'structure'}">
-      <xacro:structure_sensor name="left_rgbd_camera" parent="${name}_link" topics_ns="left_rgbd_camera">
-        <origin xyz="${left_rgbd_x} ${left_rgbd_y} ${left_rgbd_z}" rpy="${left_rgbd_R * deg_to_rad} ${left_rgbd_P * deg_to_rad} ${left_rgbd_Y * deg_to_rad}"/>
-      </xacro:structure_sensor>
-      <xacro:structure_sensor name="right_rgbd_camera" parent="${name}_link" topics_ns="right_rgbd_camera">
-        <origin xyz="${right_rgbd_x} ${right_rgbd_y} ${right_rgbd_z}" rpy="${right_rgbd_R * deg_to_rad} ${right_rgbd_P * deg_to_rad} ${right_rgbd_Y * deg_to_rad}"/>
-      </xacro:structure_sensor>
     </xacro:if>
     <xacro:base name="${name}"/>

Commit message: updated base rgbd extrinsic parameters

File: pmb3_description/urdf/base/base_pmb3_calib.urdf.xacro (robot description, xacro)
@@ -7,5 +7,5 @@
   <xacro:property name="base_rgbd_z" value="0.147644299790751"/>
   <xacro:property name="base_rgbd_R" value="21.612"/>
-  <xacro:property name="base_rgbd_P" value="29.904"/>
+  <xacro:property name="base_rgbd_P" value="31.00"/>
   <xacro:property name="roof_rgbd_z" value="0.164028397812952"/>
   <xacro:property name="roof_rgbd_R" value="180.0"/>
