Commit message: fixed/wheels slippage

File: pmb3_description/urdf/wheels/caster.urdf.xacro (robot description, xacro)
@@ -137,13 +137,8 @@
         xyz="0 0 6.17310698704775E-05"
         rpy="0 0 0" />
-      <mass
-        value="0.122536883449448" />
-      <inertia
-        ixx="5.143649657879E-05"
-        ixy="-2.55310614726917E-21"
-        ixz="4.57949223323614E-21"
-        iyy="5.143649657879E-05"
-        iyz="-1.41711420438758E-21"
-        izz="8.55807030651471E-05" />
+      <mass value="0.08855784"/>
+        <inertia  ixx="0.00001075" ixy="0" ixz="0"
+                  iyy="0.00001541" iyz="0"
+                  izz="0.00001075"/>
     </inertial>
     <visual>

File: pmb3_description/urdf/wheels/rotacaster.gazebo.xacro (robot description, xacro)
@@ -11,11 +11,11 @@
     <!-- Contact model for the rotacaster wheel surface -->
     <gazebo reference="rotacaster_${side}_link">
-      <kp>1000000.0</kp>
-      <kd>1000.0</kd>
-      <mu1>0.0</mu1>
-      <mu2>0.0</mu2>
+      <kp>100000000.0</kp>
+      <kd>10.0</kd>
+      <mu1>0.1</mu1>
+      <mu2>0.1</mu2>
       <fdir1>1 0 0</fdir1>
       <maxVel>1.0</maxVel>
-      <minDepth>0.00</minDepth>
+      <minDepth>0.0005</minDepth>
       <implicitSpringDamper>1</implicitSpringDamper>
       <material>Gazebo/DarkGrey</material>

File: pmb3_description/urdf/wheels/rotacaster.urdf.xacro (robot description, xacro)
@@ -21,5 +21,5 @@
           rpy="0 0 0" />
         <mass
-          value="44.522746198516" />
+          value="0.522746198516" />
         <inertia
           ixx="1.20266192350964"

File: pmb3_description/urdf/wheels/wheel.urdf.xacro (robot description, xacro)
@@ -19,12 +19,8 @@
       <inertial>
         <origin xyz="6.96206955455241E-05 2.26046624622056E-05 ${-0.000537771034191503 * reflect}" rpy="0 0 0"/>
-        <mass value="1.30468312314655"/>
-        <inertia
-          ixx="0.00335246532285387"
-          ixy="${-4.14934717884663E-07 * reflect}"
-          ixz="4.83252300093776E-08"
-          iyy="0.00335016326369408"
-          iyz="${1.59142713909937E-07 * reflect}"
-          izz="0.00620544284896242" />
+         <mass value="1.82362"/>
+        <inertia ixx="0.00499743171" ixy="${ 0.00000004464 * reflect}" ixz="-0.00000002245"
+          iyy="0.00499741733" iyz="${-0.00000000164 * reflect}"
+          izz="0.00839239692"/>
       </inertial>
       <visual>
