Commit message: feat: Migrate to ROS 2

File: pmb3_description/urdf/wheels/caster.gazebo.xacro (robot description, xacro)
@@ -1,51 +1,80 @@
 <?xml version="1.0"?>
 <!--
-  Copyright (c) 2022, PAL Robotics, S.L.
-  All rights reserved.
-  This work is licensed under the Creative Commons Attribution-NonCommercial-NoDerivs 3.0 Unported License.
-  To view a copy of this license, visit http://creativecommons.org/licenses/by-nc-nd/3.0/ or send a letter to
-  Creative Commons, 444 Castro Street, Suite 900, Mountain View, California, 94041, USA.
--->
-<robot xmlns:xacro="http://ros.org/wiki/xacro">
+  Copyright (c) 2023 PAL Robotics S.L. All rights reserved.
+  Licensed under the Apache License, Version 2.0 (the "License");
+  you may not use this file except in compliance with the License.
+  You may obtain a copy of the License at
+      http://www.apache.org/licenses/LICENSE-2.0
+  Unless required by applicable law or agreed to in writing, software
+  distributed under the License is distributed on an "AS IS" BASIS,
+  WITHOUT WARRANTIES OR CONDITIONS OF ANY KIND, either express or implied.
+  See the License for the specific language governing permissions and
+  limitations under the License.
+ -->
+ <robot xmlns:xacro="http://ros.org/wiki/xacro">
   <xacro:macro name="caster_gazebo" params="side">
     <!-- Contact model for the caster wheel surface -->
     <gazebo reference="caster_${side}_1_link">
       <kp>100000000.0</kp>
-      <kd>10.0</kd>
-      <mu1>0.0</mu1>
-      <mu2>0.0</mu2>
+      <kd>10000.0</kd>
+      <friction>
+        <ode>
+          <mu1>0.0</mu1>
+          <mu2>0.0</mu2>
+        </ode>
+      </friction>
       <fdir1>1 0 0</fdir1>
-      <maxVel>10.0</maxVel>
-      <minDepth>0.0005</minDepth>
+      <max_vel>1.0</max_vel>
+      <min_depth>0.005</min_depth>
       <material>Gazebo/DarkGrey</material>
     </gazebo>
     <gazebo reference="caster_${side}_2_link">
-      <kp>10000000.0</kp>
-      <kd>10.0</kd>
-      <mu1>0.0</mu1>
-      <mu2>0.0</mu2>
+      <kp>1000000.0</kp>
+      <kd>10000.0</kd>
+      <friction>
+        <ode>
+          <mu1>0.0</mu1>
+          <mu2>0.0</mu2>
+        </ode>
+      </friction>
       <fdir1>1 0 0</fdir1>
-      <maxVel>0.1</maxVel>
-      <minDepth>0.0005</minDepth>
+      <max_vel>1.0</max_vel>
+      <min_depth>0.005</min_depth>
       <material>Gazebo/DarkGrey</material>
     </gazebo>
     <gazebo reference="caster_${side}_3_link">
-      <kp>10000000.0</kp>
-      <kd>10.0</kd>
-      <mu1>0.0</mu1>
-      <mu2>0.0</mu2>
+      <kp>1000000.0</kp>
+      <kd>10000.0</kd>
+      <friction>
+        <ode>
+          <mu1>0.0</mu1>
+          <mu2>0.0</mu2>
+        </ode>
+      </friction>
       <fdir1>1 0 0</fdir1>
-      <maxVel>1.0</maxVel>
-      <minDepth>0.0005</minDepth>
+      <max_vel>1.0</max_vel>
+      <min_depth>0.005</min_depth>
       <material>Gazebo/DarkGrey</material>
     </gazebo>
     <gazebo reference="caster_{side}_1_joint">
-      <implicitSpringDamper>1</implicitSpringDamper>
+      <physics>
+        <ode>
+          <implicit_spring_damper>1</implicit_spring_damper>
+        </ode>
+      </physics>
     </gazebo>
     <gazebo reference="caster_{side}_2_joint">
-      <implicitSpringDamper>1</implicitSpringDamper>
+      <physics>
+        <ode>
+          <implicit_spring_damper>1</implicit_spring_damper>
+        </ode>
+      </physics>
     </gazebo>
     <gazebo reference="caster_{side}_3_joint">
-      <implicitSpringDamper>1</implicitSpringDamper>
+      <physics>
+        <ode>
+          <implicit_spring_damper>1</implicit_spring_damper>
+        </ode>
+      </physics>
     </gazebo>
   </xacro:macro>

File: pmb3_description/urdf/wheels/caster.urdf.xacro (robot description, xacro)
@@ -1,5 +1,5 @@
 <?xml version="1.0"?>
 <!--
-  Copyright (c) 2022 PAL Robotics S.L. All rights reserved.
+  Copyright (c) 2023 PAL Robotics S.L. All rights reserved.
   Licensed under the Apache License, Version 2.0 (the "License");
   you may not use this file except in compliance with the License.
@@ -11,5 +11,5 @@
   See the License for the specific language governing permissions and
   limitations under the License.
--->
+ -->
 <robot xmlns:xacro="http://ros.org/wiki/xacro">
   <xacro:include filename="$(find pmb3_description)/urdf/wheels/caster.gazebo.xacro"/>

File: pmb3_description/urdf/wheels/rotacaster.gazebo.xacro (robot description, xacro)
@@ -1,22 +1,35 @@
 <?xml version="1.0"?>
 <!--
-  Copyright (c) 2022, PAL Robotics, S.L.
-  All rights reserved.
-  This work is licensed under the Creative Commons Attribution-NonCommercial-NoDerivs 3.0 Unported License.
-  To view a copy of this license, visit http://creativecommons.org/licenses/by-nc-nd/3.0/ or send a letter to
-  Creative Commons, 444 Castro Street, Suite 900, Mountain View, California, 94041, USA.
--->
+  Copyright (c) 2023 PAL Robotics S.L. All rights reserved.
+  Licensed under the Apache License, Version 2.0 (the "License");
+  you may not use this file except in compliance with the License.
+  You may obtain a copy of the License at
+      http://www.apache.org/licenses/LICENSE-2.0
+  Unless required by applicable law or agreed to in writing, software
+  distributed under the License is distributed on an "AS IS" BASIS,
+  WITHOUT WARRANTIES OR CONDITIONS OF ANY KIND, either express or implied.
+  See the License for the specific language governing permissions and
+  limitations under the License.
+ -->
 <robot xmlns:xacro="http://ros.org/wiki/xacro">
   <xacro:macro name="rotacaster_gazebo" params="side">
     <!-- Contact model for the rotacaster wheel surface -->
     <gazebo reference="rotacaster_${side}_link">
-      <kp>100000000.0</kp>
-      <kd>10.0</kd>
-      <mu1>0.1</mu1>
-      <mu2>0.1</mu2>
+      <kp>1000000.0</kp>
+      <kd>10000.0</kd>
+      <friction>
+        <ode>
+          <mu1>0.1</mu1>
+          <mu2>0.1</mu2>
+        </ode>
+      </friction>
       <fdir1>1 0 0</fdir1>
-      <maxVel>1.0</maxVel>
-      <minDepth>0.0005</minDepth>
-      <implicitSpringDamper>1</implicitSpringDamper>
+      <max_vel>1.0</max_vel>
+      <min_depth>0.005</min_depth>
+      <physics>
+        <ode>
+          <implicit_spring_damper>1</implicit_spring_damper>
+        </ode>
+      </physics>
       <material>Gazebo/DarkGrey</material>
     </gazebo>

File: pmb3_description/urdf/wheels/rotacaster.urdf.xacro (robot description, xacro)
@@ -1,5 +1,5 @@
 <?xml version="1.0"?>
 <!--
-  Copyright (c) 2022 PAL Robotics S.L. All rights reserved.
+  Copyright (c) 2023 PAL Robotics S.L. All rights reserved.
   Licensed under the Apache License, Version 2.0 (the "License");
   you may not use this file except in compliance with the License.
@@ -11,5 +11,5 @@
   See the License for the specific language governing permissions and
   limitations under the License.
--->
+ -->
 <robot xmlns:xacro="http://ros.org/wiki/xacro">
   <xacro:include filename="$(find pmb3_description)/urdf/wheels/rotacaster.gazebo.xacro"/>

File: pmb3_description/urdf/wheels/wheel.gazebo.xacro (robot description, xacro)
@@ -1,10 +1,15 @@
 <?xml version="1.0"?>
 <!--
-  Copyright (c) 2022, PAL Robotics, S.L.
-  All rights reserved.
-  This work is licensed under the Creative Commons Attribution-NonCommercial-NoDerivs 3.0 Unported License.
-  To view a copy of this license, visit http://creativecommons.org/licenses/by-nc-nd/3.0/ or send a letter to
-  Creative Commons, 444 Castro Street, Suite 900, Mountain View, California, 94041, USA.
--->
+  Copyright (c) 2023 PAL Robotics S.L. All rights reserved.
+  Licensed under the Apache License, Version 2.0 (the "License");
+  you may not use this file except in compliance with the License.
+  You may obtain a copy of the License at
+      http://www.apache.org/licenses/LICENSE-2.0
+  Unless required by applicable law or agreed to in writing, software
+  distributed under the License is distributed on an "AS IS" BASIS,
+  WITHOUT WARRANTIES OR CONDITIONS OF ANY KIND, either express or implied.
+  See the License for the specific language governing permissions and
+  limitations under the License.
+ -->
 <robot xmlns:xacro="http://ros.org/wiki/xacro">
   <xacro:macro name="wheel_gazebo" params="side">
@@ -13,13 +18,21 @@
       <kp>1000000.0</kp>
       <kd>100.0</kd>
-      <mu1>100000000000000.0</mu1>
-      <mu2>100000000000000.0</mu2>
+      <friction>
+        <ode>
+          <mu>1.0</mu>
+          <mu2>1.0</mu2>
+        </ode>
+      </friction>
       <fdir1>1 0 0</fdir1>
-      <maxVel>1.0</maxVel>
-      <minDepth>0.00</minDepth>
+      <max_vel>1.0</max_vel>
+      <min_depth>0.0</min_depth>
       <material>Gazebo/DarkGrey</material>
     </gazebo>
     <gazebo reference="wheel_{side}_joint">
-      <implicitSpringDamper>1</implicitSpringDamper>
+      <physics>
+        <ode>
+          <implicit_spring_damper>1</implicit_spring_damper>
+        </ode>
+      </physics>
     </gazebo>
   </xacro:macro>
