Commit message: add support to ydlidar-tg15/tg30 and sick-561

File: pmb3_description/robots/pmb3.urdf.xacro (robot description, xacro)
@@ -8,10 +8,14 @@
 -->
 <robot  xmlns:xacro="http://ros.org/wiki/xacro" name="pmb3" >
-  <xacro:arg name="laser_model" default="sick-nanoscan-3"/> <!-- false, hokuyo, sick-551, sick-561, sick-571, sick-nanoscan-3-->
-  <xacro:arg name="camera_model" default="realsense-d435"/> <!-- false, realsense-d435, structure-->
+  <xacro:arg name="laser_model" default="ydlidar-tg30"/>
+  <xacro:arg name="camera_model" default="realsense-d435"/>
   <xacro:arg name="multiple" default="false"/>
   <xacro:arg name="namespace" default=""/>
   <xacro:property name="is_multiple" value="$(arg multiple)" />
   <xacro:property name="nsp" value="$(arg namespace)" />
+  <xacro:property name="laser_model" value="$(arg laser_model)" />
+  <xacro:if value="${laser_model not in ['No', 'false', False, 'sick-551', 'sick-561', 'sick-571', 'hokuyo', 'ydlidar-tg30', 'ydlidar-tg15']}">
+    <xacro:wrong_laser_model/>
+  </xacro:if>
   <!-- The following included files set up definitions of parts of the robot body -->
   <!-- Base -->

File: pmb3_description/urdf/base/base_sensors.urdf.xacro (robot description, xacro)
@@ -9,6 +9,9 @@
 <robot xmlns:xacro="http://ros.org/wiki/xacro">
   <xacro:include filename="$(find pmb3_description)/urdf/base/base.urdf.xacro"/>
+  <xacro:include filename="$(find pmb2_description)/urdf/sensors/sick_tim561_laser.urdf.xacro"/>
+  <xacro:include filename="$(find pmb2_description)/urdf/sensors/sick_tim571_laser.urdf.xacro"/>
   <xacro:include filename="$(find pmb3_description)/urdf/sensors/sick_nanoscan3_laser.urdf.xacro"/>
-  <xacro:include filename="$(find pmb2_description)/urdf/sensors/sick_tim571_laser.urdf.xacro"/>
+  <xacro:include filename="$(find pmb3_description)/urdf/sensors/ydlidar_tg30_laser.urdf.xacro"/>
+  <xacro:include filename="$(find pmb3_description)/urdf/sensors/ydlidar_tg15_laser.urdf.xacro"/>
   <xacro:include filename="$(find realsense2_description)/urdf/_d435.urdf.xacro" />
   <xacro:include filename="$(find pmb3_description)/urdf/deg_to_rad.xacro"/>
@@ -27,7 +30,14 @@
   <xacro:property name="roof_rgbd_y" value="0.117678395770306"/>
   <xacro:property name="roof_rgbd_Y" value="-10.0"/>
-  <!-- Laser model can be: false, hokuyo, sick-551, sick-561, sick-571, sick-nanoscan-3 -->
-  <!-- Camera model can be: false, realsense-d435, structure -->
-  <xacro:macro name="base_sensors" params=" name laser_model:=sick-nanoscan-3 camera_model:=realsense-d435">
+  <!-- Laser model can be: false, sick-561, sick-571, sick-nanoscan-3, ydlidar-tg30 -->
+  <!-- Camera model can be: false, realsense-d435 -->
+  <xacro:macro name="base_sensors" params=" name laser_model:=ydlidar-tg30 camera_model:=realsense-d435">
+    <xacro:if value="${laser_model == 'sick-561'}">
+      <!-- Laser -->
+      <!-- Theoretic FOV = 220 -->
+      <xacro:sick_tim561_laser name="${name}_laser" parent="${name}" ros_topic="scan_raw" update_rate="10" min_angle="${-110 * deg_to_rad}" max_angle="${110 * deg_to_rad}" >
+        <origin xyz="${base_laser_x} ${base_laser_y} ${base_laser_z}" rpy="0 0 0" />
+      </xacro:sick_tim561_laser>
+    </xacro:if>
     <xacro:if value="${laser_model == 'sick-571'}">
       <!-- Laser -->
@@ -44,4 +54,18 @@
       </xacro:sick_nanoscan3_laser>
     </xacro:if>
+    <xacro:if value="${laser_model == 'ydlidar-tg30'}">
+      <!-- Laser -->
+      <!-- Theoretic FOV = 360 (using 240) -->
+      <xacro:ydlidar_tg30_laser name="${name}_laser" parent="${name}" ros_topic="scan_raw" update_rate="10" min_angle="${-120 * deg_to_rad}" max_angle="${120 * deg_to_rad}" >
+        <origin xyz="${base_laser_x} ${base_laser_y} ${base_laser_z}" rpy="0 0 0" />
+      </xacro:ydlidar_tg30_laser>
+    </xacro:if>
+    <xacro:if value="${laser_model == 'ydlidar-tg15'}">
+      <!-- Laser -->
+      <!-- Theoretic FOV = 360 (using 240) -->
+      <xacro:ydlidar_tg15_laser name="${name}_laser" parent="${name}" ros_topic="scan_raw" update_rate="10" min_angle="${-120 * deg_to_rad}" max_angle="${120 * deg_to_rad}" >
+        <origin xyz="${base_laser_x} ${base_laser_y} ${base_laser_z}" rpy="0 0 0" />
+      </xacro:ydlidar_tg15_laser>
+    </xacro:if>
     <!-- RGBD camera -->
     <xacro:if value="${camera_model == 'realsense-d435'}">

Commit message: added camera_model "realsense-d435"

File: pmb3_description/robots/pmb3.urdf.xacro (robot description, xacro)
@@ -12,5 +12,7 @@
   <xacro:arg name="multiple" default="false"/>
   <xacro:arg name="namespace" default=""/>
+  <xacro:arg name="simulation" default="true" />
   <xacro:property name="is_multiple" value="$(arg multiple)" />
+  <xacro:property name="use_nominal_extrinsics" value="$(arg simulation)"/>
   <xacro:property name="nsp" value="$(arg namespace)" />
   <xacro:property name="laser_model" value="$(arg laser_model)" />

File: pmb3_description/urdf/base/base_sensors.urdf.xacro (robot description, xacro)
@@ -32,5 +32,5 @@
   <!-- Laser model can be: false, sick-561, sick-571, sick-nanoscan-3, ydlidar-tg30 -->
   <!-- Camera model can be: false, realsense-d435 -->
-  <xacro:macro name="base_sensors" params=" name laser_model:=ydlidar-tg30 camera_model:=realsense-d435">
+  <xacro:macro name="base_sensors" params=" name laser_model:=ydlidar-tg30 camera_model:=realsense-d435 ">
     <xacro:if value="${laser_model == 'sick-561'}">
       <!-- Laser -->
@@ -70,8 +70,8 @@
     <!-- RGBD camera -->
     <xacro:if value="${camera_model == 'realsense-d435'}">
-      <xacro:sensor_d435 name="roof_rgbd_camera" parent="${name}_link" topics_ns="roof_rgbd_camera">
+      <xacro:sensor_d435 name="roof_rgbd_camera" parent="${name}_link" topics_ns="roof_rgbd_camera" use_nominal_extrinsics="${use_nominal_extrinsics}">
         <origin xyz="${roof_rgbd_x} ${roof_rgbd_y} ${roof_rgbd_z}" rpy="${roof_rgbd_R * deg_to_rad} ${roof_rgbd_P * deg_to_rad} ${roof_rgbd_Y * deg_to_rad}"/>
       </xacro:sensor_d435>
-      <xacro:sensor_d435 name="base_rgbd_camera" parent="${name}_link" topics_ns="base_rgbd_camera">
+      <xacro:sensor_d435 name="base_rgbd_camera" parent="${name}_link" topics_ns="base_rgbd_camera" use_nominal_extrinsics="${use_nominal_extrinsics}">
         <origin xyz="${base_rgbd_x} ${base_rgbd_y} ${base_rgbd_z}" rpy="${base_rgbd_R * deg_to_rad} ${base_rgbd_P * deg_to_rad} ${base_rgbd_Y * deg_to_rad}"/>
       </xacro:sensor_d435>

Commit message: Set use_sim_time false as default

File: pmb3_description/robots/pmb3.urdf.xacro (robot description, xacro)
@@ -17,5 +17,5 @@
   <xacro:arg name="multiple" default="false"/>
   <xacro:arg name="namespace" default=""/>
-  <xacro:arg name="simulation" default="true" />
+  <xacro:arg name="simulation" default="false" />
   <xacro:property name="is_multiple" value="$(arg multiple)" />
   <xacro:property name="use_nominal_extrinsics" value="$(arg simulation)"/>

File: pmb3_description/ros2_control/ros2_control.urdf.xacro (robot description, xacro)
@@ -14,5 +14,5 @@
 <robot xmlns:xacro="http://ros.org/wiki/xacro"
        name="pmb3" >
-<xacro:macro name="pmb3_ros2_control" params="simulation:=^|true">
+<xacro:macro name="pmb3_ros2_control" params="simulation:=^|false">
     <xacro:include filename="$(find pmb3_description)/urdf/wheels/wheel.ros2_control.xacro"/>
     <xacro:include filename="$(find pmb3_description)/urdf/sensors/sensors.ros2_control.xacro"/>

Commit message: Rename simulation argument to use_sim

File: pmb3_description/robots/pmb3.urdf.xacro (robot description, xacro)
@@ -17,7 +17,7 @@
   <xacro:arg name="multiple" default="false"/>
   <xacro:arg name="namespace" default=""/>
-  <xacro:arg name="simulation" default="false" />
+  <xacro:arg name="use_sim" default="false" />
   <xacro:property name="is_multiple" value="$(arg multiple)" />
-  <xacro:property name="use_nominal_extrinsics" value="$(arg simulation)"/>
+  <xacro:property name="use_nominal_extrinsics" value="$(arg use_sim)"/>
   <xacro:property name="nsp" value="$(arg namespace)" />
   <xacro:property name="laser_model" value="$(arg laser_model)" />
@@ -32,5 +32,5 @@
   <!-- ros2_control -->
   <xacro:include filename="$(find pmb3_description)/ros2_control/ros2_control.urdf.xacro" />
-  <xacro:pmb3_ros2_control simulation="$(arg simulation)" />
+  <xacro:pmb3_ros2_control use_sim="$(arg use_sim)" />
   <!-- Materials for visualization -->
   <xacro:include filename="$(find pmb3_description)/urdf/materials.urdf.xacro" />

File: pmb3_description/ros2_control/ros2_control.urdf.xacro (robot description, xacro)
@@ -14,9 +14,9 @@
 <robot xmlns:xacro="http://ros.org/wiki/xacro"
        name="pmb3" >
-<xacro:macro name="pmb3_ros2_control" params="simulation:=^|false">
+<xacro:macro name="pmb3_ros2_control" params="use_sim:=^|false">
     <xacro:include filename="$(find pmb3_description)/urdf/wheels/wheel.ros2_control.xacro"/>
     <xacro:include filename="$(find pmb3_description)/urdf/sensors/sensors.ros2_control.xacro"/>
     <ros2_control name="ros2_control_pmb3_system" type="system">
-      <xacro:if value="$(arg simulation)">
+      <xacro:if value="$(arg use_sim)">
         <xacro:ros2_control_imu name="base_imu_sensor"/>
         <hardware>
@@ -24,5 +24,5 @@
         </hardware>
       </xacro:if>
-      <xacro:unless value="$(arg simulation)">
+      <xacro:unless value="$(arg use_sim)">
         <hardware>
           <plugin>robot_control/RobotControl</plugin>
